Commit message: g

File: src/rds_description/urdf/gps_marker_cybertruck.urdf.xacro (robot description, xacro)
@@ -3,8 +3,9 @@
 <!-- xmlns:xacro="http://www.ros.org/wiki/xacro" -->
   <!-- Define the base link with your STL model -->
+  <!-- 1.5708 -->
   <link name="marker_base_link">
     <visual>
     <!-- Rotate 90 degrees around X-axis -->
-      <origin xyz="0 0 0.3" rpy="1.5708 0 0" />
+      <origin xyz="-0.50 -0.50 0.3" rpy="0 0 0" />
         <geometry>
           <mesh filename="package://rds_description/meshes/full_truck.stl" scale="0.05 0.05 0.05"/>
